Commit message: updated with arm DOF

File: examples/locomotion/spot.urdf (robot description, URDF)
Before this commit: robot spot, 16 links, 15 joints
Links:
- added link arm0_link_ee
- added link arm0_link_el0; visual mesh filename=../meshes/arm0_link_el0.obj
- added link arm0_link_el1; visual mesh filename=../meshes/arm0_link_el1.obj
- added link arm0_link_fngr; visual mesh filename=../meshes/arm0_link_fngr.obj
- added link arm0_link_hr0; visual mesh filename=../meshes/arm0_link_hr0.obj
- added link arm0_link_sh0; visual mesh filename=../meshes/arm0_link_sh0.obj
- added link arm0_link_sh1; visual mesh filename=../meshes/arm0_link_sh1.obj
- added link arm0_link_wr0; visual mesh filename=../meshes/arm0_link_wr0.obj
- added link arm0_link_wr1; visual mesh filename=../meshes/arm0_link_wr1.obj
Joints:
- added joint arm0_ee_joint: type fixed, parent arm0_link_fngr, child arm0_link_ee, origin xyz=0.13 0.0 -0.06 rpy=0 0 0
- added joint arm0_el0: type revolute, parent arm0_link_hr0, child arm0_link_el0, origin xyz=0.3385 0 0 rpy=0 0 0, axis 0 1 0, limit lower=0 upper=3.14159265358979311599 effort=1000 velocity=1000.00
- added joint arm0_el1: type revolute, parent arm0_link_el0, child arm0_link_el1, origin xyz=0.40330 0.0 0.0750 rpy=0 0 0, axis 1 0 0, limit lower=-2.79252680319092716487 upper=2.79252680319092716487 effort=1000 velocity=1000.00
- added joint arm0_f1x: type revolute, parent arm0_link_wr1, child arm0_link_fngr, origin xyz=0.11745 0 0.014820 rpy=0 0 0, axis 0.0 1.0 0.0, limit lower=-1.57 upper=0.0 effort=1000 velocity=1000.00
- added joint arm0_hr0: type revolute, parent arm0_link_sh1, child arm0_link_hr0, origin xyz=0.0 0.0 0.0 rpy=0 0 0, axis 1 0 0, limit lower=-1e6 upper=1e6 effort=1000 velocity=1000.00
- added joint arm0_sh0: type fixed, parent base_link, child arm0_link_sh0, origin xyz=0.292 0.0 0.188 rpy=0 0 0, axis 0 0 1, limit lower=-2.61799387799149441136 upper=3.14159265358979311599 effort=1000 velocity=1000.00
- added joint arm0_sh1: type revolute, parent arm0_link_sh0, child arm0_link_sh1, origin xyz=0.0 0.0 0.0 rpy=0 0 0, axis 0 1 0, limit lower=-3.14159265358979311599 upper=0.52359877559829881565 effort=1000 velocity=1000.00
- added joint arm0_wr0: type revolute, parent arm0_link_el1, child arm0_link_wr0, origin xyz=0.0 0.0 0.0 rpy=0 0 0, axis 0 1 0, limit lower=-1.83259571459404613236 upper=1.83259571459404613236 effort=1000 velocity=1000.00
- added joint arm0_wr1: type revolute, parent arm0_link_wr0, child arm0_link_wr1, origin xyz=0.0 0.0 0.0 rpy=0 0 0, axis 1 0 0, limit lower=-2.87979326579064354163 upper=2.87979326579064354163 effort=1000 velocity=1000.00
